Commit message: pre-push

File: soa_description/urdf/soa_macro.xacro (robot description, xacro)
@@ -1,29 +1,13 @@
 <?xml version="1.0" encoding="utf-8"?>
-<!--
-  SOA (SO-101/SO-100) 6-DOF Robot Arm Xacro Macro
-  This macro defines a single SOA arm with parameterized prefix support for multi-arm scenarios.
-  Parameters:
-    - prefix: String prepended to all joint and link names (e.g., "left_", "right_", "")
-    - parent_link: Name of the parent link to which the arm base will be attached
-    - *origin: Transform from parent_link to arm base_link
-  Usage:
-    <xacro:soa_arm prefix="left_" parent_link="world">
-      <origin xyz="0 0 0" rpy="0 0 0"/>
-    </xacro:soa_arm>
--->
 <robot xmlns:xacro="http://www.ros.org/wiki/xacro">
-  <!-- SOA Arm Macro -->
-  <xacro:macro name="soa_arm" params="prefix parent_link *origin">
-    <!-- Common Properties -->
+  <xacro:macro name="soa" params="prefix parent_link *origin">
     <xacro:property name="effort_limit" value="10.0"/>
     <xacro:property name="velocity_limit" value="10.0"/>
     <xacro:property name="joint_damping" value="0.1"/>
     <xacro:property name="joint_friction" value="0.1"/>
-    <!-- Material Definition -->
     <material name="${prefix}yellow">
       <color rgba="1.0 1.0 0.0 1.0"/>
     </material>
     <!-- ========== LINKS ========== -->
-    <!-- Base Link -->
     <link name="${prefix}base_link">
       <inertial>
@@ -33,5 +17,4 @@
                  iyy="0.000136117" iyz="9.75275e-08" izz="0.000130364"/>
       </inertial>
-      <!-- Base motor holder -->
       <visual>
         <origin xyz="-0.00636471 -9.94414e-05 -0.0024" rpy="1.5708 -1.67685e-15 1.5708"/>
@@ -47,5 +30,4 @@
         </geometry>
       </collision>
-      <!-- Base platform -->
       <visual>
         <origin xyz="-0.00636471 -8.97657e-09 -0.0024" rpy="1.5708 -2.78073e-29 1.5708"/>
@@ -61,5 +43,4 @@
         </geometry>
       </collision>
-      <!-- Servo (shoulder pan motor) -->
       <visual>
         <origin xyz="0.0263353 -8.97657e-09 0.0437" rpy="-8.21148e-16 7.84513e-18 1.249e-15"/>
@@ -75,5 +56,4 @@
         </geometry>
       </collision>
-      <!-- Mounting plate -->
       <visual>
         <origin xyz="-0.0309827 -0.000199441 0.0474" rpy="1.5708 -1.35493e-14 1.5708"/>
@@ -90,5 +70,4 @@
       </collision>
     </link>
-    <!-- Shoulder Link -->
     <link name="${prefix}shoulder_link">
       <inertial>
@@ -98,5 +77,4 @@
                  iyy="8.10403e-05" iyz="1.54663e-07" izz="2.39783e-05"/>
       </inertial>
-      <!-- Servo (shoulder lift motor) -->
       <visual>
         <origin xyz="-0.0303992 0.000422241 -0.0417" rpy="1.5708 1.5708 0"/>
@@ -112,5 +90,4 @@
         </geometry>
       </collision>
-      <!-- Motor holder (base/shoulder) -->
       <visual>
         <origin xyz="-0.0675992 -0.000177759 0.0158499" rpy="1.5708 -1.5708 0"/>
@@ -126,5 +103,4 @@
         </geometry>
       </collision>
-      <!-- Rotation pitch mechanism -->
       <visual>
         <origin xyz="0.0122008 2.22413e-05 0.0464" rpy="-1.5708 2.35221e-33 0"/>
@@ -141,5 +117,4 @@
       </collision>
     </link>
-    <!-- Upper Arm Link -->
     <link name="${prefix}upper_arm_link">
       <inertial>
@@ -149,5 +124,4 @@
                  iyy="0.000147318" iyz="8.97326e-09" izz="0.000142487"/>
       </inertial>
-      <!-- Servo (elbow motor) -->
       <visual>
         <origin xyz="-0.11257 -0.0155 0.0187" rpy="-3.14159 -5.27356e-16 -1.5708"/>
@@ -163,5 +137,4 @@
         </geometry>
       </collision>
-      <!-- Upper arm structure -->
       <visual>
         <origin xyz="-0.065085 0.012 0.0182" rpy="3.14159 -0 -1.30911e-30"/>
@@ -178,5 +151,4 @@
       </collision>
     </link>
-    <!-- Lower Arm Link (Forearm) -->
     <link name="${prefix}lower_arm_link">
       <inertial>
@@ -186,5 +158,4 @@
                  iyy="0.000159844" iyz="-4.90188e-08" izz="0.00014529"/>
       </inertial>
-      <!-- Lower arm (forearm) structure -->
       <visual>
         <origin xyz="-0.0648499 -0.032 0.0182" rpy="3.14159 -0 6.67202e-31"/>
@@ -200,5 +171,4 @@
         </geometry>
       </collision>
-      <!-- Wrist motor holder -->
       <visual>
         <origin xyz="-0.0648499 -0.032 0.018" rpy="-3.14159 -2.55351e-15 -1.83387e-30"/>
@@ -214,5 +184,4 @@
         </geometry>
       </collision>
-      <!-- Servo (wrist flex motor) -->
       <visual>
         <origin xyz="-0.1224 0.0052 0.0187" rpy="-3.14159 -7.88861e-31 -3.14159"/>
@@ -229,5 +198,4 @@
       </collision>
     </link>
-    <!-- Wrist Link -->
     <link name="${prefix}wrist_link">
       <inertial>
@@ -237,5 +205,4 @@
                  iyy="2.5391e-05" iyz="3.6412e-06" izz="2.1e-05"/>
       </inertial>
-      <!-- Servo (wrist roll motor, no horn) -->
       <visual>
         <origin xyz="8.32667e-17 -0.0424 0.0306" rpy="1.5708 1.5708 0"/>
@@ -251,5 +218,4 @@
         </geometry>
       </collision>
-      <!-- Wrist roll/pitch assembly -->
       <visual>
         <origin xyz="0 -0.028 0.0181" rpy="-1.5708 -1.5708 0"/>
@@ -266,5 +232,4 @@
       </collision>
     </link>
-    <!-- Gripper Link -->
     <link name="${prefix}gripper_link">
       <inertial>
@@ -274,5 +239,4 @@
                  iyy="4.33657e-05" iyz="-5.17847e-08" izz="3.45059e-05"/>
       </inertial>
-      <!-- Servo (gripper motor) -->
       <visual>
         <origin xyz="0.0077 0.0001 -0.0234" rpy="-1.5708 -5.19179e-17 -1.66533e-16"/>
@@ -288,5 +252,4 @@
         </geometry>
       </collision>
-      <!-- Wrist roll follower -->
       <visual>
         <origin xyz="8.32667e-17 -0.000218214 0.000949706" rpy="-3.14159 -5.55112e-17 0"/>
@@ -303,5 +266,4 @@
       </collision>
     </link>
-    <!-- Gripper Frame (TCP - Tool Center Point) -->
     <link name="${prefix}gripper_frame_link">
       <inertial>
@@ -311,5 +273,4 @@
       </inertial>
     </link>
-    <!-- Moving Jaw Link -->
     <link name="${prefix}moving_jaw_link">
       <inertial>
@@ -319,5 +280,4 @@
                  iyy="1.89032e-06" iyz="-1.09945e-07" izz="5.28738e-06"/>
       </inertial>
-      <!-- Moving jaw -->
       <visual>
         <origin xyz="-5.55112e-17 -5.55112e-17 0.0189" rpy="9.53145e-17 6.93889e-18 1.24077e-24"/>
@@ -335,5 +295,4 @@
     </link>
     <!-- ========== JOINTS ========== -->
-    <!-- Joint: Parent Link to Base Link -->
     <joint name="${prefix}base_joint" type="fixed">
       <xacro:insert_block name="origin"/>
@@ -341,5 +300,4 @@
       <child link="${prefix}base_link"/>
     </joint>
-    <!-- Joint: Shoulder Pan (Base Rotation) -->
     <joint name="${prefix}shoulder_pan" type="revolute">
       <origin xyz="0.0388353 -8.97657e-09 0.0624" rpy="3.14159 4.18253e-17 -3.14159"/>
@@ -350,5 +308,4 @@
       <dynamics damping="${joint_damping}" friction="${joint_friction}"/>
     </joint>
-    <!-- Joint: Shoulder Lift -->
     <joint name="${prefix}shoulder_lift" type="revolute">
       <origin xyz="-0.0303992 -0.0182778 -0.0542" rpy="-1.5708 -1.5708 0"/>
@@ -359,5 +316,4 @@
       <dynamics damping="${joint_damping}" friction="${joint_friction}"/>
     </joint>
-    <!-- Joint: Elbow Flex -->
     <joint name="${prefix}elbow_flex" type="revolute">
       <origin xyz="-0.11257 -0.028 1.73763e-16" rpy="-3.63608e-16 8.74301e-16 1.5708"/>
@@ -368,5 +324,4 @@
       <dynamics damping="${joint_damping}" friction="${joint_friction}"/>
     </joint>
-    <!-- Joint: Wrist Flex -->
     <joint name="${prefix}wrist_flex" type="revolute">
       <origin xyz="-0.1349 0.0052 3.62355e-17" rpy="4.02456e-15 8.67362e-16 -1.5708"/>
@@ -377,5 +332,4 @@
       <dynamics damping="${joint_damping}" friction="${joint_friction}"/>
     </joint>
-    <!-- Joint: Wrist Roll -->
     <joint name="${prefix}wrist_roll" type="revolute">
       <origin xyz="5.55112e-17 -0.0611 0.0181" rpy="1.5708 0.0486795 3.14159"/>
@@ -386,5 +340,4 @@
       <dynamics damping="${joint_damping}" friction="${joint_friction}"/>
     </joint>
-    <!-- Joint: Gripper (Jaw Open/Close) -->
     <joint name="${prefix}gripper" type="revolute">
       <origin xyz="0.0202 0.0188 -0.0234" rpy="1.5708 -5.24284e-08 -1.41553e-15"/>
@@ -395,5 +348,4 @@
       <dynamics damping="${joint_damping}" friction="${joint_friction}"/>
     </joint>
-    <!-- Joint: Gripper Frame (Fixed TCP) -->
     <joint name="${prefix}gripper_frame_joint" type="fixed">
       <origin xyz="-0.0079 -0.000218121 -0.0981274" rpy="0 3.14159 0"/>

Commit message: remove param joint in base xacro macro

File: soa_description/urdf/soa_macro.xacro (robot description, xacro)
@@ -1,5 +1,5 @@
 <?xml version="1.0" encoding="utf-8"?>
 <robot xmlns:xacro="http://www.ros.org/wiki/xacro">
-  <xacro:macro name="soa" params="prefix parent_link *origin">
+  <xacro:macro name="soa" params="prefix">
     <xacro:property name="effort_limit" value="10.0"/>
     <xacro:property name="velocity_limit" value="10.0"/>
@@ -295,9 +295,4 @@
     </link>
     <!-- ========== JOINTS ========== -->
-    <joint name="${prefix}base_joint" type="fixed">
-      <xacro:insert_block name="origin"/>
-      <parent link="${parent_link}"/>
-      <child link="${prefix}base_link"/>
-    </joint>
     <joint name="${prefix}shoulder_pan" type="revolute">
       <origin xyz="0.0388353 -8.97657e-09 0.0624" rpy="3.14159 4.18253e-17 -3.14159"/>

Commit message: expand joint limits

File: soa_description/urdf/soa_macro.xacro (robot description, xacro)
@@ -300,5 +300,5 @@
       <child link="${prefix}shoulder_link"/>
       <axis xyz="0 0 1"/>
-      <limit effort="${effort_limit}" velocity="${velocity_limit}" lower="-1.91986" upper="1.91986"/>
+      <limit effort="${effort_limit}" velocity="${velocity_limit}" lower="-2.04786" upper="2.04786"/>
       <dynamics damping="${joint_damping}" friction="${joint_friction}"/>
     </joint>
@@ -308,5 +308,5 @@
       <child link="${prefix}upper_arm_link"/>
       <axis xyz="0 0 1"/>
-      <limit effort="${effort_limit}" velocity="${velocity_limit}" lower="-1.74533" upper="1.74533"/>
+      <limit effort="${effort_limit}" velocity="${velocity_limit}" lower="-1.89089" upper="1.89089"/>
       <dynamics damping="${joint_damping}" friction="${joint_friction}"/>
     </joint>
@@ -316,5 +316,5 @@
       <child link="${prefix}lower_arm_link"/>
       <axis xyz="0 0 1"/>
-      <limit effort="${effort_limit}" velocity="${velocity_limit}" lower="-1.69" upper="1.69"/>
+      <limit effort="${effort_limit}" velocity="${velocity_limit}" lower="-1.69021" upper="1.69021"/>
       <dynamics damping="${joint_damping}" friction="${joint_friction}"/>
     </joint>
@@ -324,5 +324,5 @@
       <child link="${prefix}wrist_link"/>
       <axis xyz="0 0 1"/>
-      <limit effort="${effort_limit}" velocity="${velocity_limit}" lower="-1.65806" upper="1.65806"/>
+      <limit effort="${effort_limit}" velocity="${velocity_limit}" lower="-1.78913" upper="1.78913"/>
       <dynamics damping="${joint_damping}" friction="${joint_friction}"/>
     </joint>
@@ -332,5 +332,5 @@
       <child link="${prefix}gripper_link"/>
       <axis xyz="0 0 1"/>
-      <limit effort="${effort_limit}" velocity="${velocity_limit}" lower="-2.74385" upper="2.84121"/>
+      <limit effort="${effort_limit}" velocity="${velocity_limit}" lower="-2.99306" upper="2.99306"/>
       <dynamics damping="${joint_damping}" friction="${joint_friction}"/>
     </joint>
@@ -340,5 +340,5 @@
       <child link="${prefix}moving_jaw_link"/>
       <axis xyz="0 0 1"/>
-      <limit effort="${effort_limit}" velocity="${velocity_limit}" lower="-0.174533" upper="1.74533"/>
+      <limit effort="${effort_limit}" velocity="${velocity_limit}" lower="-0.28839" upper="1.85050"/>
       <dynamics damping="${joint_damping}" friction="${joint_friction}"/>
     </joint>
