Commit message: stand urdf

File: soa_description/urdf/bi_soa.urdf.xacro (robot description, xacro)
@@ -34,11 +34,19 @@
   <xacro:include filename="$(find soa_description)/urdf/soa_macro.xacro"/>
   <xacro:include filename="$(find soa_description)/urdf/soa_ros2_control.xacro"/>
+  <xacro:include filename="$(find soa_description)/urdf/stand.xacro"/>
   <!-- Shared root link -->
   <link name="base_link"/>
-  <!-- Left arm: +Y from center -->
+  <!-- Stand -->
+  <joint name="base_to_stand" type="fixed">
+    <parent link="base_link"/>
+    <child link="stand_link"/>
+    <origin xyz="0 0 0" rpy="0 0 0"/>
+  </joint>
+  <xacro:stand/>
+  <!-- Left arm: -Y from center -->
   <joint name="left_base_joint" type="fixed">
     <parent link="base_link"/>
     <child link="left_base_link"/>
-    <origin xyz="0 0.15 0" rpy="0 0 0"/>
+    <origin xyz="-0.01775 -0.13575 0.0248" rpy="0 0 0"/>
   </joint>
   <xacro:soa prefix="left_"/>
@@ -61,9 +69,9 @@
     gripper_id="$(arg left_gripper_id)"
     gripper_offset="$(arg left_gripper_offset)"/>
-  <!-- Right arm: -Y from center -->
+  <!-- Right arm: +Y from center -->
   <joint name="right_base_joint" type="fixed">
     <parent link="base_link"/>
     <child link="right_base_link"/>
-    <origin xyz="0 -0.15 0" rpy="0 0 0"/>
+    <origin xyz="-0.01775 0.13575 0.0248" rpy="0 0 0"/>
   </joint>
   <xacro:soa prefix="right_"/>

File: soa_description/urdf/bi_soa_kinematics.urdf.xacro (robot description, xacro)
@@ -2,18 +2,26 @@
 <robot xmlns:xacro="http://www.ros.org/wiki/xacro" name="bi_soa">
   <xacro:include filename="$(find soa_description)/urdf/soa_macro.xacro"/>
+  <xacro:include filename="$(find soa_description)/urdf/stand.xacro"/>
   <!-- Shared root link -->
   <link name="base_link"/>
-  <!-- Left arm: +Y from center -->
+  <!-- Stand -->
+  <joint name="base_to_stand" type="fixed">
+    <parent link="base_link"/>
+    <child link="stand_link"/>
+    <origin xyz="0 0 0" rpy="0 0 0"/>
+  </joint>
+  <xacro:stand/>
+  <!-- Left arm: -Y from center -->
   <joint name="left_base_joint" type="fixed">
     <parent link="base_link"/>
     <child link="left_base_link"/>
-    <origin xyz="0 0.15 0" rpy="0 0 0"/>
+    <origin xyz="-0.01775 -0.13575 0.0248" rpy="0 0 0"/>
   </joint>
   <xacro:soa prefix="left_"/>
-  <!-- Right arm: -Y from center -->
+  <!-- Right arm: +Y from center -->
   <joint name="right_base_joint" type="fixed">
     <parent link="base_link"/>
     <child link="right_base_link"/>
-    <origin xyz="0 -0.15 0" rpy="0 0 0"/>
+    <origin xyz="-0.01775 0.13575 0.0248" rpy="0 0 0"/>
   </joint>
   <xacro:soa prefix="right_"/>

Commit message: bi soa moveit config

File: soa_description/urdf/bi_soa.urdf.xacro (robot description, xacro)
@@ -44,9 +44,9 @@
   </joint>
   <xacro:stand/>
-  <!-- Left arm: -Y from center -->
+  <!-- Left arm: +Y from center -->
   <joint name="left_base_joint" type="fixed">
     <parent link="base_link"/>
     <child link="left_base_link"/>
-    <origin xyz="-0.01775 -0.13575 0.0248" rpy="0 0 0"/>
+    <origin xyz="-0.01775 0.13575 0.0248" rpy="0 0 0"/>
   </joint>
   <xacro:soa prefix="left_"/>
@@ -69,9 +69,9 @@
     gripper_id="$(arg left_gripper_id)"
     gripper_offset="$(arg left_gripper_offset)"/>
-  <!-- Right arm: +Y from center -->
+  <!-- Right arm: -Y from center -->
   <joint name="right_base_joint" type="fixed">
     <parent link="base_link"/>
     <child link="right_base_link"/>
-    <origin xyz="-0.01775 0.13575 0.0248" rpy="0 0 0"/>
+    <origin xyz="-0.01775 -0.13575 0.0248" rpy="0 0 0"/>
   </joint>
   <xacro:soa prefix="right_"/>

File: soa_description/urdf/bi_soa_kinematics.urdf.xacro (robot description, xacro)
@@ -12,16 +12,16 @@
   </joint>
   <xacro:stand/>
-  <!-- Left arm: -Y from center -->
+  <!-- Left arm: +Y from center -->
   <joint name="left_base_joint" type="fixed">
     <parent link="base_link"/>
     <child link="left_base_link"/>
-    <origin xyz="-0.01775 -0.13575 0.0248" rpy="0 0 0"/>
+    <origin xyz="-0.01775 0.13575 0.0248" rpy="0 0 0"/>
   </joint>
   <xacro:soa prefix="left_"/>
-  <!-- Right arm: +Y from center -->
+  <!-- Right arm: -Y from center -->
   <joint name="right_base_joint" type="fixed">
     <parent link="base_link"/>
     <child link="right_base_link"/>
-    <origin xyz="-0.01775 0.13575 0.0248" rpy="0 0 0"/>
+    <origin xyz="-0.01775 -0.13575 0.0248" rpy="0 0 0"/>
   </joint>
   <xacro:soa prefix="right_"/>
